File: rs485-uart.kicad_pcb (KiCad board)
At the start: 2 copper layers, 40 x 20 mm, 8 parts, among them J1 Conn_01x06, J2 Conn_01x06, U1 ISL83490IBZ

Commit message: Tuning
Other:
- board text added: "←TX"
- board text added: "→RX"
- board text removed: "RX"
- board text removed: "TX"
Changed lines of the file:
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@@
 			(sketchpadsonfab no)
 			(subtractmaskfromsilk no)
-			(outputformat 1)
+			(outputformat 4)
 			(mirror no)
-			(drillshape 1)
+			(drillshape 0)
 			(scaleselection 1)
-			(outputdirectory "")
+			(outputdirectory "outputs/")
 		)
 	)
@@
 		)
 	)
-	(gr_text "RX"
+	(gr_text "→RX"
 		(at 133.5 71.909 0)
 		(layer "F.SilkS")
@@
 		)
 	)
-	(gr_text "RX"
+	(gr_text "→RX"
 		(at 133.5 74.449 0)
 		(layer "F.SilkS")
@@
 		)
 	)
-	(gr_text "TX"
+	(gr_text "←TX"
 		(at 133.5 69.369 0)
 		(layer "F.SilkS")
@@
 		)
 	)
-	(gr_text "TX"
+	(gr_text "←TX"
 		(at 133.5 66.829 0)
 		(layer "F.SilkS")
